File: pcb/linesnifferbot.sch (KiCad schematic (older format))
At the start: 73 parts

Commit message: More or less finalized schematic and First version of PCB
Parts:
- removed J? (x2): GS2, Connectors:GS2, symbol GS2
- removed Q?: Q_NMOS_DGS, symbol Q_NMOS_DGS
- removed R? (x2): 0R18, symbol R
- removed R? (x4): 10k, symbol R
- removed U? (x2): DRV8870, symbol DRV8870
- added C1: 10uF, Capacitors_SMD:C_1206, symbol C_Small
- added C10, C12, C4, C7, C8, C9: 100nF, Capacitors_SMD:C_0805, symbol C_Small
- added C2: 10nF, Capacitors_SMD:C_0805, symbol C_Small
- added C3: 2.2uF, Capacitors_SMD:C_0805, symbol C_Small
- added J10: CONN_01X09, Socket_Strips:Socket_Strip_Straight_1x09_Pitch2.54mm, symbol CONN_01X09
- added J7: CONN_01X06, Socket_Strips:Socket_Strip_Straight_1x06_Pitch2.54mm, symbol CONN_01X06
- added Q1: Q_NMOS_GSD, TO_SOT_Packages_SMD:SOT-23, symbol Q_NMOS_GSD
- added R21: 10k, Resistors_SMD:R_0805, symbol R
- added R22: DNP, Resistors_SMD:R_0805, symbol R
- added U1: DRV8833, Housings_SSOP:TSSOP-16_4.4x5mm_Pitch0.65mm, symbol DRV8833
- BT1: renamed from BT?; footprint (none) -> Footprints:RN-42
- BT2: renamed from BT?; footprint (none) -> Footprints:PP3Battery
- C11, C13, C14: renamed from C?; footprint (none) -> Capacitors_Tantalum_SMD:CP_Tantalum_Case-A_EIA-3216-18_Reflow
- C5, C6: renamed from C?; footprint (none) -> Capacitors_SMD:C_0805
- D1, D2, D5: renamed from D?; footprint (none) -> LEDs:LED_0805
- D3: renamed from D?; value STATUS -> ST2; footprint (none) -> LEDs:LED_0805
- D4: renamed from D?; value STATUS -> ST1; footprint (none) -> LEDs:LED_0805
- J3: renamed from J?; value GS3 -> RxSel; footprint Connectors:GS3 -> Connect:GS3
- J4: renamed from J?; value GS3 -> TxSel; footprint Connectors:GS3 -> Connect:GS3
- J5: renamed from J?; value GS3 -> IntSelA; footprint Connectors:GS3 -> Connect:GS3
- J6: renamed from J?; value GS3 -> IntSelB; footprint Connectors:GS3 -> Connect:GS3
- J8: renamed from J?; value GS2 -> Btn2EN; footprint Connectors:GS2 -> Connect:GS2
- J9: renamed from J?; value GS2 -> LED2EN; footprint Connectors:GS2 -> Connect:GS2
- JP1, JP2: renamed from JP?; footprint (none) -> Connect:GS2
- ME1, ME2: renamed from ME?; footprint (none) -> Footprints:PololuMotoEncoder
- R1, R10, R11, R12, R13, R14, R15, R16, R17, R18, R19, R2, R20, R4, R5, R7, R9: renamed from R?; footprint (none) -> Resistors_SMD:R_0805
- R3: renamed from R?; value 10k -> 20k; footprint (none) -> Resistors_SMD:R_0805
- R6: renamed from R?; value R -> 0R02; footprint (none) -> Resistors_SMD:R_1206
- R8: renamed from R?; value 10k -> 25k; footprint (none) -> Resistors_SMD:R_0805
- S1, S2, S3, S4, S5, S6, S7, S8: renamed from S?; footprint (none) -> Footprints:QRE1113GR
- SW1: renamed from SW?; footprint (none) -> Footprints:SP_ToggleSW
- SW2: renamed from SW?; value BTN -> BTN2; footprint (none) -> Buttons_Switches_SMD:SW_SPST_EVPBF
- SW3: renamed from SW?; value BTN -> BTN1; footprint (none) -> Buttons_Switches_SMD:SW_SPST_EVPBF
- U10: renamed from U?; footprint (none) -> TO_SOT_Packages_SMD:SOT-223
- U2, U3: renamed from U?; footprint (none) -> Housings_SOIC:SOIC-14_3.9x8.7mm_Pitch1.27mm
- U4, U5, U7: renamed from U?; footprint (none) -> TO_SOT_Packages_SMD:SOT-23-5
- U6: renamed from U?; footprint (none) -> Footprints:ArduinoMicro
- U8: renamed from U?; footprint (none) -> Footprints:DPAK3
- U9: renamed from U?; footprint (none) -> Housings_SOIC:SOIC-16_3.9x9.9mm_Pitch1.27mm
Connections:
- net I2C_SCL_3.3V is gone; now on an unnamed net: U2.2 (A1)
- net I2C_SDA_3.3V is gone; now on an unnamed net: U2.3 (A2)
- net +3V3: now also J7.5 (P5)
- net +5V: now also C12.2, C4.1, C7.1, C8.1, J7.4 (P4)
- net +9V: now also C1.2, C2.2, J7.1 (P1), U1.1 (nSLEEP), U1.12 (VM)
- net GND: now also C1.1, C10.2, C12.1, C3.1, C4.2, C7.2, C8.2, C9.2, J10.9 (P9), J7.2 (P2), J7.3 (P3), J7.6 (P6), Q1.2 (S), U1.13 (GND), U1.3 (AISEN), U1.6 (BISEN)
- net at U6.14 (9(PWM)/A9): now also U1.15 (AIN2)
- net at U6.15 (10(PWM)/A10): now also U1.16 (AIN1)
- net at ME1.1 (M1): now also U1.2 (AOUT1)
- net at ME1.2 (M2): now also U1.4 (AOUT2)
- net at U6.10 (5(PWM)): now also U1.10 (BIN2)
- net at U6.11 (6(PWM)/A7): now also U1.9 (BIN1)
- net at ME2.1 (M1): now also U1.7 (BOUT1)
- net at ME2.2 (M2): now also U1.5 (BOUT2)
- net SPI_MOSI: now reaches U6.1 (MOSI)
- net SPI_MOSI: now also J10.3 (P3)
- net IO7(INT): now reaches J3.1 (G1), J8.1 (G1), U6.12 (7(INT))
- net IO7(INT): now also J10.7 (P7)
- net IO8/A8: now reaches J4.1 (G1), J9.1 (G1), U6.13 (8/A8)
- net IO8/A8: now also J10.8 (P8)
- net SPI_SS: now reaches U6.2 (RX_L/SS)
- net SPI_SS: now also J10.4 (P4)
- net at R8.1, U7.1 (OUT): now also C10.1, R21.1; no longer U6.25 (A4)
- net at R3.2, R4.1: now also U6.25 (A4), C9.1; no longer U6.26 (A5)
- net SPI_MISO: now reaches U6.33 (MISO)
- net SPI_MISO: now also J10.2 (P2)
- net SPI_CLK: now reaches U6.34 (SCK)
- net SPI_CLK: now also J10.1 (P1)
- net I2C_SDA: now reaches J5.1 (G1), U6.7 (2(INT)/SDA)
- net I2C_SDA: now also J10.5 (P5)
- net I2C_SCL: now reaches J6.1 (G1), U6.8 (3(PWM,INT)/SCL)
- net I2C_SCL: now also J10.6 (P6)
- net at U6.9 (4/A6): now also Q1.1 (G)
- net at S3.2, S6.2, S8.2: now also Q1.3 (D)
- net I2C_SCL_5V: no longer names the net of U2.13 (B1)
- net I2C_SCL_5V: now also R22.1
- net I2C_SDA_5V: no longer names the net of U2.12 (B2)
- net I2C_SDA_5V: now also R22.2
- new net: R21.2, U6.26 (A5)
- new net: C2.1, U1.11 (VCP)
- new net: C3.2, U1.14 (VINT)
- no-connect marks 30 -> 26
Other:
- note added: "Addon headers"
- note added: "Communication"
- note added: "Line sensors"
- note added: "Microcontroler"
- note added: "Motor and encoder support circuits"
- note added: "Power supply"
- moved on the sheet: BT2, C11, C13, C14, D5, J8, ME1, ME2, R3, R4, R6, R8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
